Commit message: simplified models

File: ws/src/franka_description/robots/old/panda.urdf.xacro (robot description, xacro)
@@ -11,4 +11,5 @@
   <!-- spawn robot -->
   <xacro:panda_arm />
+  <!-- <xacro:panda_hand ns="panda" rpy="0 0 ${-pi/4}" connected_to="panda_link8"/> -->
   <xacro:panda_gazebo robot_name="$(arg robot_name)" />
   <xacro:panda_transmission robot_name="$(arg robot_name)" />

File: ws/src/franka_description/robots/old/panda_arm.xacro (robot description, xacro)
@@ -3,5 +3,13 @@
   <!--: Minimum safety distance [m] by which the collision volumes are expanded and which is enforced during robot motions -->
   <!-- arm_id: Namespace of the panda arm. Serves to differentiate between arms in case of multiple instances. -->
-  <xacro:macro name="panda_arm" params="arm_id:='panda' package_name:='franka_description' xyz:='0 0 0' rpy:='0 0 0' joint_damping='1.0'">
+  <xacro:macro name="panda_arm" params="arm_id:='panda' package_name:='franka_description' connected_to:='' xyz:='0 0 0' rpy:='0 0 0' joint_damping='1.0'">
+    <!-- ??? -->
+    <xacro:unless value="${not connected_to}">
+      <joint name="${arm_id}_joint_${connected_to}" type="fixed">
+        <parent link="${connected_to}"/>
+        <child link="${arm_id}_link0"/>
+        <origin rpy="${rpy}" xyz="${xyz}"/>
+      </joint>
+    </xacro:unless>
     <!-- fix the robot to the Gazebo world coordinate system  -->
     <link name="world" />
