Commit message: added new dynamic parameters

File: ws/src/franka_description/robots/panda_arm.old.xacro (robot description, xacro)
@@ -3,13 +3,5 @@
   <!--: Minimum safety distance [m] by which the collision volumes are expanded and which is enforced during robot motions -->
   <!-- arm_id: Namespace of the panda arm. Serves to differentiate between arms in case of multiple instances. -->
-  <xacro:macro name="panda_arm" params="arm_id:='panda' package_name:='franka_description' connected_to:='' xyz:='0 0 0' rpy:='0 0 0' joint_damping='1.0'">
-    <!-- ??? -->
-    <xacro:unless value="${not connected_to}">
-      <joint name="${arm_id}_joint_${connected_to}" type="fixed">
-        <parent link="${connected_to}"/>
-        <child link="${arm_id}_link0"/>
-        <origin rpy="${rpy}" xyz="${xyz}"/>
-      </joint>
-    </xacro:unless>
+  <xacro:macro name="panda_arm" params="arm_id:='panda' package_name:='franka_description' xyz:='0 0 0' rpy:='0 0 0' joint_damping='1.0'">
     <!-- fix the robot to the Gazebo world coordinate system  -->
     <link name="world" />

File: ws/src/franka_description/robots/panda_arm.xacro (robot description, xacro)
@@ -15,7 +15,7 @@
     <link name="${arm_id}_link0">
       <inertial>
-        <mass value="2.92" />
+        <mass value="1.937868" />
         <origin xyz="-0.025566 -2.88e-05 0.057332" rpy="0 0 0" />
-        <inertia ixx="0.00782229414331" ixy="-1.56191622996e-05" ixz="-0.00126005738123" iyy="0.0109027971813" iyz="1.08233858202e-05" izz="0.0102355503949" />
+        <inertia ixx="1" ixy="0" ixz="0" iyy="1" iyz="0" izz="1" />
       </inertial>
       <visual>
@@ -38,7 +38,7 @@
     <link name="${arm_id}_link1">
       <inertial>
-        <mass value="2.74" />
+        <mass value="4.970684" />
         <origin xyz="0 -0.0324958 -0.0675818" rpy="0 0 0" />
-        <inertia ixx="0.0180416958283" ixy="0.0" ixz="0.0" iyy="0.0159136071891" iyz="0.0046758424612" izz="0.00620690827127" />
+        <inertia ixx="0.551121276649726" ixy="-9.891702555950000e-05" ixz="0.003401254912500" iyy="0.554308164573063" iyz="0.017358801154300" izz="0.009020836222789"/>
       </inertial>
       <visual>
@@ -70,7 +70,7 @@
     <link name="${arm_id}_link2">
       <inertial>
-        <mass value="2.74" />
+        <mass value="0.646926"/>
         <origin xyz="0 -0.06861 0.0322285" rpy="0 0 0" />
-        <inertia ixx="0.0182856182281" ixy="0.0" ixz="0.0" iyy="0.00621358421175" iyz="-0.00472844221905" izz="0.0161514346309" />
+        <inertia ixx="0.007420488375978" ixy="-0.003866641116064" ixz="0.010246898178992" iyy="0.028095715287805" iyz="6.390638970536000e-04" izz="0.025455008098310"/>
       </inertial>
       <visual>
@@ -102,7 +102,7 @@
     <link name="${arm_id}_link3">
       <inertial>
-        <mass value="2.38" />
+        <mass value="3.228604"/>
         <origin xyz="0.0469893 0.0316374 -0.031704" rpy="0 0 0" />
-        <inertia ixx="0.00771376630908" ixy="-0.00248490625138" ixz="-0.00332147581033" iyy="0.00989108008727" iyz="-0.00217796151484" izz="0.00811723558464" />
+        <inertia ixx="0.017989073985929" ixy="-0.001273666859324" ixz="-0.017304351893438" iyy="0.019431618000394" iyz="-0.021232742878160" izz="0.003410797707480"/>
       </inertial>
       <visual>
@@ -134,7 +134,7 @@
     <link name="${arm_id}_link4">
       <inertial>
-        <mass value="2.38" />
+        <mass value="3.587895"/>
         <origin xyz="-0.0360446 0.0336853 0.031882" rpy="0 0 0" />
-        <inertia ixx="0.00799663881132" ixy="0.00347095570217" ixz="-0.00241222942995" iyy="0.00825390705278" iyz="0.00235774044121" izz="0.0102515004345" />
+        <inertia ixx="-0.015971270250860" ixy="-0.012123843173626" ixz="-0.006569355026276" iyy="0.006704569575549" iyz="0.018926487577369" izz="-0.020940149052540"/>
       </inertial>
       <visual>
@@ -166,7 +166,7 @@
     <link name="${arm_id}_link5">
       <inertial>
-        <mass value="2.74" />
+        <mass value="1.225946"/>
         <origin xyz="0 0.0610427 -0.104176" rpy="0 0 0" />
-        <inertia ixx="0.030371374513" ixy="6.50283587108e-07" ixz="-1.05129179916e-05" iyy="0.0288752887402" iyz="-0.00775653445787" izz="0.00444134056164" />
+        <inertia ixx="0.031670429041964" ixy="-0.002718755526673" ixz="-0.003473754482437" iyy="0.027487627674740" iyz="-0.001706052052098" izz="0.006384489237171"/>
       </inertial>
       <visual>
@@ -198,7 +198,7 @@
     <link name="${arm_id}_link6">
       <inertial>
-        <mass value="1.55" />
+        <mass value="1.666555"/>
         <origin xyz="0.0510509 0.009108 0.0106343" rpy="0 0 0" />
-        <inertia ixx="0.00303336450376" ixy="-0.000437276865508" ixz="0.000629257294877" iyy="0.00404479911567" iyz="0.000130472021025" izz="0.00558234286039" />
+        <inertia ixx="0.001447539641829" ixy="-0.001306110902883" ixz="-0.002212241082781" iyy="-0.001859766133107" iyz="5.884309026853950e-04" izz="-9.285602302389487e-04"/>
       </inertial>
       <visual>
@@ -230,7 +230,7 @@
     <link name="${arm_id}_link7">
       <inertial>
-        <mass value="0.54" />
+        <mass value="7.35522e-01"/>
         <origin xyz="0.0109695 0.0107965 0.0650411" rpy="0 0 0" />
-        <inertia ixx="0.000888868887021" ixy="-0.00012239074652" ixz="3.98699829666e-05" iyy="0.000888001373233" iyz="-9.33825115206e-05" izz="0.0007176834609" />
+        <inertia ixx="0.009711991609050" ixy="-4.608912816842480e-04" ixz="-7.195173382162220e-04" iyy="0.007154935387572" iyz="-9.336408935917680e-04" izz="0.004720348032639"/>
       </inertial>
       <visual>
