Commit message: fix dynamic parameters

File: ws/src/franka_description/robots/panda_arm.xacro (robot description, xacro)
@@ -38,6 +38,6 @@
     <link name="${arm_id}_link1">
       <inertial>
-        <mass value="4.970684" />
-        <origin xyz="0 -0.0324958 -0.0675818" rpy="0 0 0" />
+        <origin xyz="3.875e-03 2.081e-03 -0.1750" rpy="0 0 0"/>
+        <mass value="4.970684"/>
         <inertia ixx="0.551121276649726" ixy="-9.891702555950000e-05" ixz="0.003401254912500" iyy="0.554308164573063" iyz="0.017358801154300" izz="0.009020836222789"/>
       </inertial>
@@ -70,6 +70,6 @@
     <link name="${arm_id}_link2">
       <inertial>
+        <origin xyz="-3.141e-03 -2.872e-02 3.495e-03" rpy="0 0 0"/>
         <mass value="0.646926"/>
-        <origin xyz="0 -0.06861 0.0322285" rpy="0 0 0" />
         <inertia ixx="0.007420488375978" ixy="-0.003866641116064" ixz="0.010246898178992" iyy="0.028095715287805" iyz="6.390638970536000e-04" izz="0.025455008098310"/>
       </inertial>
@@ -102,6 +102,6 @@
     <link name="${arm_id}_link3">
       <inertial>
+        <origin xyz="2.7518e-02 3.9252e-02 -6.6502e-02" rpy="0 0 0"/>
         <mass value="3.228604"/>
-        <origin xyz="0.0469893 0.0316374 -0.031704" rpy="0 0 0" />
         <inertia ixx="0.017989073985929" ixy="-0.001273666859324" ixz="-0.017304351893438" iyy="0.019431618000394" iyz="-0.021232742878160" izz="0.003410797707480"/>
       </inertial>
@@ -134,6 +134,6 @@
     <link name="${arm_id}_link4">
       <inertial>
+        <origin xyz="-5.317e-02 1.04419e-01 2.7454e-02" rpy="0 0 0"/>
         <mass value="3.587895"/>
-        <origin xyz="-0.0360446 0.0336853 0.031882" rpy="0 0 0" />
         <inertia ixx="-0.015971270250860" ixy="-0.012123843173626" ixz="-0.006569355026276" iyy="0.006704569575549" iyz="0.018926487577369" izz="-0.020940149052540"/>
       </inertial>
@@ -166,6 +166,6 @@
     <link name="${arm_id}_link5">
       <inertial>
+        <origin xyz="-1.1953e-02 4.1065e-02 -3.8437e-02" rpy="0 0 0"/>
         <mass value="1.225946"/>
-        <origin xyz="0 0.0610427 -0.104176" rpy="0 0 0" />
         <inertia ixx="0.031670429041964" ixy="-0.002718755526673" ixz="-0.003473754482437" iyy="0.027487627674740" iyz="-0.001706052052098" izz="0.006384489237171"/>
       </inertial>
@@ -198,6 +198,6 @@
     <link name="${arm_id}_link6">
       <inertial>
+        <origin xyz="6.0149e-02 -1.4117e-02 -1.0517e-02" rpy="0 0 0"/>
         <mass value="1.666555"/>
-        <origin xyz="0.0510509 0.009108 0.0106343" rpy="0 0 0" />
         <inertia ixx="0.001447539641829" ixy="-0.001306110902883" ixz="-0.002212241082781" iyy="-0.001859766133107" iyz="5.884309026853950e-04" izz="-9.285602302389487e-04"/>
       </inertial>
@@ -230,6 +230,6 @@
     <link name="${arm_id}_link7">
       <inertial>
+        <origin xyz="1.0517e-02 -4.252e-03 6.1597e-02" rpy="0 0 0"/>
         <mass value="7.35522e-01"/>
-        <origin xyz="0.0109695 0.0107965 0.0650411" rpy="0 0 0" />
         <inertia ixx="0.009711991609050" ixy="-4.608912816842480e-04" ixz="-7.195173382162220e-04" iyy="0.007154935387572" iyz="-9.336408935917680e-04" izz="0.004720348032639"/>
       </inertial>

Commit message: experiments

File: ws/src/franka_description/robots/panda_arm.xacro (robot description, xacro)
@@ -3,5 +3,5 @@
   <!--: Minimum safety distance [m] by which the collision volumes are expanded and which is enforced during robot motions -->
   <!-- arm_id: Namespace of the panda arm. Serves to differentiate between arms in case of multiple instances. -->
-  <xacro:macro name="panda_arm" params="arm_id:='panda' package_name:='franka_description' xyz:='0 0 0' rpy:='0 0 0' joint_damping='1.0'">
+  <xacro:macro name="panda_arm" params="arm_id:='panda' package_name:='franka_description' xyz:='0 0 0' rpy:='0 0 0' joint_damping='0'">
     <!-- fix the robot to the Gazebo world coordinate system  -->
     <link name="world" />
@@ -59,10 +59,11 @@
     </link>
     <joint name="${arm_id}_joint1" type="revolute">
-      <safety_controller k_position="100.0" k_velocity="40.0" soft_lower_limit="-2.8973" soft_upper_limit="2.8973"/>
+      <!-- <safety_controller k_position="100.0" k_velocity="40.0" soft_lower_limit="-2.8973" soft_upper_limit="2.8973"/> -->
       <origin rpy="0 0 0" xyz="0 0 0.333"/>
       <parent link="${arm_id}_link0"/>
       <child link="${arm_id}_link1"/>
       <axis xyz="0 0 1"/>
-      <limit effort="87" lower="-2.8973" upper="2.8973" velocity="2.1750"/>
+      <limit effort="1000000000000" lower="-2.8973" upper="2.8973" velocity="1000000000000"/>
+      <!-- <limit effort="87" lower="-2.8973" upper="2.8973" velocity="2.1750"/> -->
       <dynamics damping="${joint_damping}"/>
     </joint>
@@ -91,10 +92,11 @@
     </link>
     <joint name="${arm_id}_joint2" type="revolute">
-      <safety_controller k_position="100.0" k_velocity="40.0" soft_lower_limit="-1.7628" soft_upper_limit="1.7628"/>
+      <!-- <safety_controller k_position="100.0" k_velocity="40.0" soft_lower_limit="-1.7628" soft_upper_limit="1.7628"/> -->
       <origin rpy="${-pi/2} 0 0" xyz="0 0 0"/>
       <parent link="${arm_id}_link1"/>
       <child link="${arm_id}_link2"/>
       <axis xyz="0 0 1"/>
-      <limit effort="87" lower="-1.7628" upper="1.7628" velocity="2.1750"/>
+      <limit effort="1000000000000" lower="-1.7628" upper="1.7628" velocity="1000000000000"/>
+      <!-- <limit effort="87" lower="-1.7628" upper="1.7628" velocity="2.1750"/> -->
       <dynamics damping="${joint_damping}"/>
     </joint>
@@ -123,10 +125,11 @@
     </link>
     <joint name="${arm_id}_joint3" type="revolute">
-      <safety_controller k_position="100.0" k_velocity="40.0" soft_lower_limit="-2.8973" soft_upper_limit="2.8973"/>
+      <!-- <safety_controller k_position="100.0" k_velocity="40.0" soft_lower_limit="-2.8973" soft_upper_limit="2.8973"/> -->
       <origin rpy="${pi/2} 0 0" xyz="0 -0.316 0"/>
       <parent link="${arm_id}_link2"/>
       <child link="${arm_id}_link3"/>
       <axis xyz="0 0 1"/>
-      <limit effort="87" lower="-2.8973" upper="2.8973" velocity="2.1750"/>
+      <limit effort="1000000000000" lower="-2.8973" upper="2.8973" velocity="1000000000000"/>
+      <!-- <limit effort="87" lower="-2.8973" upper="2.8973" velocity="2.1750"/> -->
       <dynamics damping="${joint_damping}"/>
     </joint>
@@ -155,10 +158,11 @@
     </link>
     <joint name="${arm_id}_joint4" type="revolute">
-      <safety_controller k_position="100.0" k_velocity="40.0" soft_lower_limit="-3.0718" soft_upper_limit="-0.0698"/>
+      <!-- <safety_controller k_position="100.0" k_velocity="40.0" soft_lower_limit="-3.0718" soft_upper_limit="-0.0698"/> -->
       <origin rpy="${pi/2} 0 0" xyz="0.0825 0 0"/>
       <parent link="${arm_id}_link3"/>
       <child link="${arm_id}_link4"/>
       <axis xyz="0 0 1"/>
-      <limit effort="87" lower="-3.0718" upper="-0.0698" velocity="2.1750"/>
+      <limit effort="1000000000000" lower="-3.0718" upper="-0.0698" velocity="1000000000000"/>
+      <!-- <limit effort="87" lower="-3.0718" upper="-0.0698" velocity="2.1750"/> -->
       <dynamics damping="${joint_damping}"/>
     </joint>
@@ -187,10 +191,11 @@
     </link>
     <joint name="${arm_id}_joint5" type="revolute">
-      <safety_controller k_position="100.0" k_velocity="40.0" soft_lower_limit="-2.8973" soft_upper_limit="2.8973"/>
+      <!-- <safety_controller k_position="100.0" k_velocity="40.0" soft_lower_limit="-2.8973" soft_upper_limit="2.8973"/> -->
       <origin rpy="${-pi/2} 0 0" xyz="-0.0825 0.384 0"/>
       <parent link="${arm_id}_link4"/>
       <child link="${arm_id}_link5"/>
       <axis xyz="0 0 1"/>
-      <limit effort="12" lower="-2.8973" upper="2.8973" velocity="2.6100"/>
+      <limit effort="1000000000000" lower="-2.8973" upper="2.8973" velocity="1000000000000"/>
+      <!-- <limit effort="12" lower="-2.8973" upper="2.8973" velocity="2.6100"/> -->
       <dynamics damping="${joint_damping}"/>
     </joint>
@@ -219,10 +224,11 @@
     </link>
     <joint name="${arm_id}_joint6" type="revolute">
-      <safety_controller k_position="100.0" k_velocity="40.0" soft_lower_limit="-0.0175" soft_upper_limit="3.7525"/>
+      <!-- <safety_controller k_position="100.0" k_velocity="40.0" soft_lower_limit="-0.0175" soft_upper_limit="3.7525"/> -->
       <origin rpy="${pi/2} 0 0" xyz="0 0 0"/>
       <parent link="${arm_id}_link5"/>
       <child link="${arm_id}_link6"/>
       <axis xyz="0 0 1"/>
-      <limit effort="12" lower="-0.0175" upper="3.7525" velocity="2.6100"/>
+      <limit effort="1000000000000" lower="-0.0175" upper="3.7525" velocity="1000000000000"/>
+      <!-- <limit effort="12" lower="-0.0175" upper="3.7525" velocity="2.6100"/> -->
       <dynamics damping="${joint_damping}"/>
     </joint>
@@ -251,10 +257,11 @@
     </link>
     <joint name="${arm_id}_joint7" type="revolute">
-      <safety_controller k_position="100.0" k_velocity="40.0" soft_lower_limit="-2.8973" soft_upper_limit="2.8973"/>
+      <!-- <safety_controller k_position="100.0" k_velocity="40.0" soft_lower_limit="-2.8973" soft_upper_limit="2.8973"/> -->
       <origin rpy="${pi/2} 0 0" xyz="0.088 0 0"/>
       <parent link="${arm_id}_link6"/>
       <child link="${arm_id}_link7"/>
       <axis xyz="0 0 1"/>
-      <limit effort="12" lower="-2.8973" upper="2.8973" velocity="2.6100"/>
+      <limit effort="1000000000000" lower="-2.8973" upper="2.8973" velocity="1000000000000"/>
+      <!-- <limit effort="12" lower="-2.8973" upper="2.8973" velocity="2.6100"/> -->
       <dynamics damping="${joint_damping}"/>
     </joint>

Commit message: revert temporary changes for Gazebo vs OpenSim comparison

File: ws/src/franka_description/robots/panda_arm.xacro (robot description, xacro)
@@ -3,5 +3,5 @@
   <!--: Minimum safety distance [m] by which the collision volumes are expanded and which is enforced during robot motions -->
   <!-- arm_id: Namespace of the panda arm. Serves to differentiate between arms in case of multiple instances. -->
-  <xacro:macro name="panda_arm" params="arm_id:='panda' package_name:='franka_description' xyz:='0 0 0' rpy:='0 0 0' joint_damping='0'">
+  <xacro:macro name="panda_arm" params="arm_id:='panda' package_name:='franka_description' xyz:='0 0 0' rpy:='0 0 0' joint_damping='1.0'">
     <!-- fix the robot to the Gazebo world coordinate system  -->
     <link name="world" />
@@ -59,11 +59,11 @@
     </link>
     <joint name="${arm_id}_joint1" type="revolute">
-      <!-- <safety_controller k_position="100.0" k_velocity="40.0" soft_lower_limit="-2.8973" soft_upper_limit="2.8973"/> -->
+      <safety_controller k_position="100.0" k_velocity="40.0" soft_lower_limit="-2.8973" soft_upper_limit="2.8973"/>
       <origin rpy="0 0 0" xyz="0 0 0.333"/>
       <parent link="${arm_id}_link0"/>
       <child link="${arm_id}_link1"/>
       <axis xyz="0 0 1"/>
-      <limit effort="1000000000000" lower="-2.8973" upper="2.8973" velocity="1000000000000"/>
-      <!-- <limit effort="87" lower="-2.8973" upper="2.8973" velocity="2.1750"/> -->
+      <!-- <limit effort="1000000000000" lower="-2.8973" upper="2.8973" velocity="1000000000000"/> -->
+      <limit effort="87" lower="-2.8973" upper="2.8973" velocity="2.1750"/>
       <dynamics damping="${joint_damping}"/>
     </joint>
@@ -92,5 +92,5 @@
     </link>
     <joint name="${arm_id}_joint2" type="revolute">
-      <!-- <safety_controller k_position="100.0" k_velocity="40.0" soft_lower_limit="-1.7628" soft_upper_limit="1.7628"/> -->
+      <safety_controller k_position="100.0" k_velocity="40.0" soft_lower_limit="-1.7628" soft_upper_limit="1.7628"/>
       <origin rpy="${-pi/2} 0 0" xyz="0 0 0"/>
       <parent link="${arm_id}_link1"/>
@@ -98,5 +98,5 @@
       <axis xyz="0 0 1"/>
       <limit effort="1000000000000" lower="-1.7628" upper="1.7628" velocity="1000000000000"/>
-      <!-- <limit effort="87" lower="-1.7628" upper="1.7628" velocity="2.1750"/> -->
+      <limit effort="87" lower="-1.7628" upper="1.7628" velocity="2.1750"/>
       <dynamics damping="${joint_damping}"/>
     </joint>
@@ -125,11 +125,11 @@
     </link>
     <joint name="${arm_id}_joint3" type="revolute">
-      <!-- <safety_controller k_position="100.0" k_velocity="40.0" soft_lower_limit="-2.8973" soft_upper_limit="2.8973"/> -->
+      <safety_controller k_position="100.0" k_velocity="40.0" soft_lower_limit="-2.8973" soft_upper_limit="2.8973"/>
       <origin rpy="${pi/2} 0 0" xyz="0 -0.316 0"/>
       <parent link="${arm_id}_link2"/>
       <child link="${arm_id}_link3"/>
       <axis xyz="0 0 1"/>
-      <limit effort="1000000000000" lower="-2.8973" upper="2.8973" velocity="1000000000000"/>
-      <!-- <limit effort="87" lower="-2.8973" upper="2.8973" velocity="2.1750"/> -->
+      <!-- <limit effort="1000000000000" lower="-2.8973" upper="2.8973" velocity="1000000000000"/> -->
+      <limit effort="87" lower="-2.8973" upper="2.8973" velocity="2.1750"/>
       <dynamics damping="${joint_damping}"/>
     </joint>
@@ -158,5 +158,5 @@
     </link>
     <joint name="${arm_id}_joint4" type="revolute">
-      <!-- <safety_controller k_position="100.0" k_velocity="40.0" soft_lower_limit="-3.0718" soft_upper_limit="-0.0698"/> -->
+      <safety_controller k_position="100.0" k_velocity="40.0" soft_lower_limit="-3.0718" soft_upper_limit="-0.0698"/>
       <origin rpy="${pi/2} 0 0" xyz="0.0825 0 0"/>
       <parent link="${arm_id}_link3"/>
@@ -164,5 +164,5 @@
       <axis xyz="0 0 1"/>
       <limit effort="1000000000000" lower="-3.0718" upper="-0.0698" velocity="1000000000000"/>
-      <!-- <limit effort="87" lower="-3.0718" upper="-0.0698" velocity="2.1750"/> -->
+      <limit effort="87" lower="-3.0718" upper="-0.0698" velocity="2.1750"/>
       <dynamics damping="${joint_damping}"/>
     </joint>
@@ -191,11 +191,11 @@
     </link>
     <joint name="${arm_id}_joint5" type="revolute">
-      <!-- <safety_controller k_position="100.0" k_velocity="40.0" soft_lower_limit="-2.8973" soft_upper_limit="2.8973"/> -->
+      <safety_controller k_position="100.0" k_velocity="40.0" soft_lower_limit="-2.8973" soft_upper_limit="2.8973"/>
       <origin rpy="${-pi/2} 0 0" xyz="-0.0825 0.384 0"/>
       <parent link="${arm_id}_link4"/>
       <child link="${arm_id}_link5"/>
       <axis xyz="0 0 1"/>
-      <limit effort="1000000000000" lower="-2.8973" upper="2.8973" velocity="1000000000000"/>
-      <!-- <limit effort="12" lower="-2.8973" upper="2.8973" velocity="2.6100"/> -->
+      <!-- <limit effort="1000000000000" lower="-2.8973" upper="2.8973" velocity="1000000000000"/> -->
+      <limit effort="12" lower="-2.8973" upper="2.8973" velocity="2.6100"/>
       <dynamics damping="${joint_damping}"/>
     </joint>
@@ -224,5 +224,5 @@
     </link>
     <joint name="${arm_id}_joint6" type="revolute">
-      <!-- <safety_controller k_position="100.0" k_velocity="40.0" soft_lower_limit="-0.0175" soft_upper_limit="3.7525"/> -->
+      <safety_controller k_position="100.0" k_velocity="40.0" soft_lower_limit="-0.0175" soft_upper_limit="3.7525"/>
       <origin rpy="${pi/2} 0 0" xyz="0 0 0"/>
       <parent link="${arm_id}_link5"/>
@@ -230,5 +230,5 @@
       <axis xyz="0 0 1"/>
       <limit effort="1000000000000" lower="-0.0175" upper="3.7525" velocity="1000000000000"/>
-      <!-- <limit effort="12" lower="-0.0175" upper="3.7525" velocity="2.6100"/> -->
+      <limit effort="12" lower="-0.0175" upper="3.7525" velocity="2.6100"/>
       <dynamics damping="${joint_damping}"/>
     </joint>
@@ -257,11 +257,11 @@
     </link>
     <joint name="${arm_id}_joint7" type="revolute">
-      <!-- <safety_controller k_position="100.0" k_velocity="40.0" soft_lower_limit="-2.8973" soft_upper_limit="2.8973"/> -->
+      <safety_controller k_position="100.0" k_velocity="40.0" soft_lower_limit="-2.8973" soft_upper_limit="2.8973"/>
       <origin rpy="${pi/2} 0 0" xyz="0.088 0 0"/>
       <parent link="${arm_id}_link6"/>
       <child link="${arm_id}_link7"/>
       <axis xyz="0 0 1"/>
-      <limit effort="1000000000000" lower="-2.8973" upper="2.8973" velocity="1000000000000"/>
-      <!-- <limit effort="12" lower="-2.8973" upper="2.8973" velocity="2.6100"/> -->
+      <!-- <limit effort="1000000000000" lower="-2.8973" upper="2.8973" velocity="1000000000000"/> -->
+      <limit effort="12" lower="-2.8973" upper="2.8973" velocity="2.6100"/>
       <dynamics damping="${joint_damping}"/>
     </joint>
